File: Readable_Schema/120VDC Treadmill Motor Controller/120VDC Treadmill Motor Controller.kicad_pcb (KiCad board)
At the start: 4 copper layers, 250.8 x 133.2 mm, 145 parts, among them J1 TB005-762-03BE, J2 OSTT7020150, J3 TB0011-350-08BE, J4 TB0011-350-08BE, J5 TB0011-350-08BE, J6 TB0011-350-03BE, J7 OSTT7020150, J9 OSTT7020150, K1 T9GV1L14-24, Q1 IPP60R060P7XKSA1, Q2 IPP60R060P7XKSA1, Q3 IPP60R060P7XKSA1, Q4 IPP60R060P7XKSA1, Q5 IPP60R060P7XKSA1, Q7 DN2450N8-G, Q8 VOM1271T, U1 UCC21530DWKR, U2 UCC21530DWKR, U3 TMCS1126B42QDVGRQ1, U4 SN74HCS08DYYR, U5 TPSI3050QDWZRQ1, U6 AMC1311BDWVR

Commit message: -Playing around with different layouts --With the additional two layers the GND and 5V planes can be shared amongst all LV components, making things a bit easier and pushing me to really start laying a bunch of SMD components one on top of the other.
Parts:
- removed NT1, NT2, NT3, NT4: NetTie_2, NetTie:NetTie-2_THT_Pad0.3mm
- C22, C23, C28, C32, C49, C50, C51, C52, C53, C54, R24, R27: moved to B.Cu
- moved U6 270.5 mm to (74.0, 113.0)
- moved R27 259.3 mm to (78.8, 147.1), turned to -90 degrees
- moved C22 257.8 mm to (74.0, 147.1), turned to 90 degrees
- moved C23 254.8 mm to (76.5, 147.1), turned to -90 degrees
- moved R24 254.2 mm to (80.8, 148.4), turned to 90 degrees
- moved R25 252.7 mm to (78.0, 122.9), turned to 90 degrees
- moved R28 249.6 mm to (80.2, 122.9), turned to 90 degrees
- moved C24 247.3 mm to (75.8, 122.9), turned to 90 degrees
- moved U5 241.1 mm to (77.8, 131.2), turned to -90 degrees
- moved TP2 201.9 mm to (55.1, 162.2)
- moved TP1 191.3 mm to (61.4, 162.2)
- moved J9 157.6 mm to (114.2, 170.8), turned to 0 degrees
- moved D3 90.8 mm to (19.2, 149.5), turned to 0 degrees
- moved C14 87.6 mm to (105.7, 145.3)
- moved Q3 85.8 mm to (26.6, 152.5), turned to 180 degrees
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Connections:
- C10 pad 2: Net-(U2-VSSB) -> /Feedback/in+
- C18 pad 1: Net-(C18-Pad1) -> Net-(J2-Pin_2)
- C19 pad 2: Net-(C18-Pad1) -> Net-(J2-Pin_2)
- C20 pad 2: Net-(U1-VSSB) -> /Feedback/in+
- C26 pad 1: Net-(C18-Pad1) -> Net-(J2-Pin_2)
- C35 pad 2: Net-(U2-VSSB) -> /Feedback/in+
- C43 pad 2: Net-(U1-VSSB) -> /Feedback/in+
- CR1 pad 1: Net-(C18-Pad1) -> Net-(J2-Pin_2)
- PS1 pad 10: unconnected-(PS1-+Vout-Pad10) -> /H_Bridge/hs_ps_1_+
- PS1 pad 16: unconnected-(PS1-+Vin-Pad16) -> 5v 15w
- PS1 pad 6: unconnected-(PS1--Vout-Pad6) -> /H_Bridge/hs_ps_1_-
- PS1 pad 8: unconnected-(PS1--Vin-Pad8) -> LV_GND
- PS2 pad 10: unconnected-(PS2-+Vout-Pad10) -> /H_Bridge/ls_ps_+
- PS2 pad 16: unconnected-(PS2-+Vin-Pad16) -> 5v 15w
- PS2 pad 6: unconnected-(PS2--Vout-Pad6) -> HV_GND
- PS2 pad 8: unconnected-(PS2--Vin-Pad8) -> LV_GND
- PS3 pad 10: unconnected-(PS3-+Vout-Pad10) -> /H_Bridge/hs_ps_2_+
- PS3 pad 16: unconnected-(PS3-+Vin-Pad16) -> 5v 15w
- PS3 pad 6: unconnected-(PS3--Vout-Pad6) -> /H_Bridge/hs_ps_2_-
- PS3 pad 8: unconnected-(PS3--Vin-Pad8) -> LV_GND
- R17 pad 1: Net-(U2-VSSB) -> /Feedback/in+
- R32 pad 1: Net-(U1-VSSB) -> /Feedback/in+
- R7 pad 2: Net-(C18-Pad1) -> Net-(J2-Pin_2)
- U1 pad 9: Net-(U1-VSSB) -> /Feedback/in+
- U2 pad 9: Net-(U2-VSSB) -> /Feedback/in+
Routing:
- net LV_GND: track 60.8 -> 0.00 mm
- net /H_Bridge/EN_drive: track 39.6 -> 0.00 mm
- net Net-(U2-INB): track 21.2 -> 0.00 mm
- net Net-(U2-INA): track 12.4 -> 0.00 mm
- net Net-(U1-INA): track 11.6 -> 0.00 mm
- net unconnected-(U2-VCCI_2-Pad8): track 6.71 -> 0.00 mm
- net Net-(U1-INB): track 5.80 -> 0.00 mm
- net 5v 15w: track 5.67 -> 0.00 mm
- net Net-(U1-DT): track 4.46 -> 0.00 mm
- net Net-(U2-DT): track 4.40 -> 0.00 mm
- net /H_Bridge/pwm_b: track 2.28 -> 0.00 mm
- net /H_Bridge/dir_a: track 2.25 -> 0.00 mm
- net /H_Bridge/pwm_a: track 2.00 -> 0.00 mm
- net /H_Bridge/dir_b: track 2.00 -> 0.00 mm
Other:
- outline, holes or cut-outs redrawn
